File: Circuit_microPowerModule/microcontroller_unit.kicad_sch (KiCad schematic)
At the start: 69 parts, among them J201 USB_C_Receptacle_USB2.0, J202 Debug, SW201 KMR2, U201 W25Q128JVS, U202 RP2040, Y201 12MHz

Commit message: Finishing MCU Peripheral Passive Components
Parts:
- added U204: USBLC6-2P6, Package_TO_SOT_SMD:SOT-666, symbol Power_Protection:USBLC6-2P6
Connections:
- net GNDREF: now also U204.2 (GND)
- net USB_N: now also U204.1 (I/O1); no longer R?.2
- net USB_P: now also U204.3 (I/O2); no longer R?.2
- net VBUS: now also U204.5 (VBUS)
- new net USB+: R?.2, U204.4 (I/O2)
- new net USB-: R?.2, U204.6 (I/O1)
Changed lines of the file:
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@@
     (stroke (width 0) (type default))
   )
+  (wire (pts (xy 60.325 55.245) (xy 67.31 55.245))
+    (stroke (width 0) (type default))
+  )
   (wire (pts (xy 146.05 38.735) (xy 146.05 36.195))
     (stroke (width 0) (type default))
@@
     (stroke (width 0) (type default))
   )
+  (wire (pts (xy 87.63 55.245) (xy 94.615 55.245))
+    (stroke (width 0) (type default))
+  )
   (wire (pts (xy 154.94 113.665) (xy 144.78 113.665))
     (stroke (width 0) (type default))
@@
     (stroke (width 0) (type default))
   )
+  (wire (pts (xy 87.63 60.325) (xy 94.615 60.325))
+    (stroke (width 0) (type default))
+  )
+  (wire (pts (xy 60.325 60.325) (xy 67.31 60.325))
+    (stroke (width 0) (type default))
+  )
   (wire (pts (xy 154.94 24.13) (xy 146.05 24.13))
     (stroke (width 0) (type default))
@@
     (effects (font (size 1.27 1.27)) (justify left bottom))
   )
-  (label "USB_P" (at 135.89 75.565 0) (fields_autoplaced)
+  (label "USB+" (at 135.89 75.565 0) (fields_autoplaced)
     (effects (font (size 1.27 1.27)) (justify left bottom))
   )
@@
     (effects (font (size 1.27 1.27)) (justify right bottom))
   )
-  (label "USB_N" (at 135.89 78.105 0) (fields_autoplaced)
+  (label "USB-" (at 135.89 78.105 0) (fields_autoplaced)
     (effects (font (size 1.27 1.27)) (justify left bottom))
   )
@@
     (effects (font (size 1.27 1.27)) (justify right bottom))
   )
+  (label "USB-" (at 60.325 55.245 0) (fields_autoplaced)
+    (effects (font (size 1.27 1.27)) (justify left bottom))
+  )
   (label "SWCLK" (at 147.32 133.985 0) (fields_autoplaced)
     (effects (font (size 1.27 1.27)) (justify left bottom))
@@
     (effects (font (size 1.27 1.27)) (justify right bottom))
   )
+  (label "USB_P" (at 94.615 60.325 180) (fields_autoplaced)
+    (effects (font (size 1.27 1.27)) (justify right bottom))
+  )
   (label "QSPI_SD3" (at 72.39 121.92 180) (fields_autoplaced)
     (effects (font (size 1.27 1.27)) (justify right bottom))
@@
     (effects (font (size 1.27 1.27)) (justify right bottom))
   )
+  (label "USB_N" (at 60.325 60.325 0) (fields_autoplaced)
+    (effects (font (size 1.27 1.27)) (justify left bottom))
+  )
   (label "~{USB}_P" (at 147.32 75.565 0) (fields_autoplaced)
     (effects (font (size 1.27 1.27)) (justify left bottom))
@@
     (effects (font (size 1.27 1.27)) (justify right bottom))
   )
+  (label "USB+" (at 94.615 55.245 180) (fields_autoplaced)
+    (effects (font (size 1.27 1.27)) (justify right bottom))
+  )
   (label "QSPI_SD3" (at 130.81 98.425 0) (fields_autoplaced)
     (effects (font (size 1.27 1.27)) (justify left bottom))
@@
     )
   )
+  (symbol (lib_id "Power_Protection:USBLC6-2P6") (at 77.47 57.785 0) (unit 1)
+    (in_bom yes) (on_board yes) (dnp no) (fields_autoplaced)
+    (property "Reference" "U204" (at 79.1211 45.72 0)
+      (effects (font (size 1.27 1.27)) (justify left))
+    )
+    (property "Value" "USBLC6-2P6" (at 79.1211 48.26 0)
+      (effects (font (size 1.27 1.27)) (justify left))
+    )
+    (property "Footprint" "Package_TO_SOT_SMD:SOT-666" (at 77.47 70.485 0)
+      (effects (font (size 1.27 1.27)) hide)
+    )
+    (property "Datasheet" "https://www.st.com/resource/en/datasheet/usblc6-2.pdf" (at 82.55 48.895 0)
+      (effects (font (size 1.27 1.27)) hide)
+    )
+    (pin "1")
+    (pin "2")
+    (pin "3")
+    (pin "4")
+    (pin "5")
+    (pin "6")
+    (instances
+      (project "micro-PowerModule"
+        (path "/38b19d1a-a8d3-49c0-a6a2-bee4e845832f/7187d72d-86a6-4df3-a706-10f93237b261"
+          (reference "U204") (unit 1)
+        )
+      )
+    )
+  )
   (symbol (lib_id "Device:C_Small") (at 207.645 29.21 0) (mirror y) (unit 1)
     (in_bom yes) (on_board yes) (dnp no)
@@
     )
   )
+  (symbol (lib_id "power:GNDREF") (at 77.47 67.945 0) (unit 1)
+    (in_bom yes) (on_board yes) (dnp no) (fields_autoplaced)
+    (property "Reference" "#PWR0221" (at 77.47 74.295 0)
+      (effects (font (size 1.27 1.27)) hide)
+    )
+    (property "Value" "GNDREF" (at 77.47 72.898 0)
+      (effects (font (size 1.27 1.27)))
+    )
+    (property "Footprint" "" (at 77.47 67.945 0)
+      (effects (font (size 1.27 1.27)) hide)
+    )
+    (property "Datasheet" "" (at 77.47 67.945 0)
+      (effects (font (size 1.27 1.27)) hide)
+    )
+    (pin "1")
+    (instances
+      (project "micro-PowerModule"
+        (path "/38b19d1a-a8d3-49c0-a6a2-bee4e845832f/7187d72d-86a6-4df3-a706-10f93237b261"
+          (reference "#PWR0221") (unit 1)
+        )
+      )
+    )
+  )
   (symbol (lib_id "Device:R_Small_US") (at 152.4 93.345 270) (unit 1)
     (in_bom yes) (on_board yes) (dnp no)
@@
         )
       )
+    )
+  )
+  (symbol (lib_id "power:VBUS") (at 77.47 47.625 0) (unit 1)
+    (in_bom yes) (on_board yes) (dnp no) (fields_autoplaced)
+    (property "Reference" "#PWR0220" (at 77.47 51.435 0)
+      (effects (font (size 1.27 1.27)) hide)
+    )
+    (property "Value" "VBUS" (at 77.47 43.307 0)
+      (effects (font (size 1.27 1.27)))
+    )
+    (property "Footprint" "" (at 77.47 47.625 0)
+      (effects (font (size 1.27 1.27)) hide)
+    )
+    (property "Datasheet" "" (at 77.47 47.625 0)
+      (effects (font (size 1.27 1.27)) hide)
+    )
+    (pin "1")
+    (instances
+      (project "micro-PowerModule"
+        (path "/38b19d1a-a8d3-49c0-a6a2-bee4e845832f/7187d72d-86a6-4df3-a706-10f93237b261"
+          (reference "#PWR0220") (unit 1)
+        )
+      )

Commit message: update system power circuit layout
Parts:
- J202: footprint Connector_PinHeader_2.54mm:PinHeader_1x03_P2.54mm_Vertical -> Connector_PinHeader_2.54mm:PinHeader_1x03_P2.54mm_Horizontal
Changed lines of the file:
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@@
       (effects (font (size 1.27 1.27)) (justify right))
     )
-    (property "Footprint" "Connector_PinHeader_2.54mm:PinHeader_1x03_P2.54mm_Vertical" (at 130.81 141.605 0)
+    (property "Footprint" "Connector_PinHeader_2.54mm:PinHeader_1x03_P2.54mm_Horizontal" (at 130.81 141.605 0)
       (effects (font (size 1.27 1.27)) hide)
     )
